File: sirin-clone-mcu.brd (EAGLE design)
At the start: 101.6 x 57.1 mm, 11 parts, among them J1 PJ-002A, J2 SWITCHCRAFT_PHONEJACK, J3 30_PIN_CONNECTOR_MALE

Commit message: routing
Parts:
- removed J2: SWITCHCRAFT_PHONEJACK, sirin-clone-library:STEREO_JACK_2SWITCH
- added C10, C14, C27, C28, C29, C3, C35, C8, C9: 0.1UF, moon-germs-v1_main:C_0805
- added C11, C12: 22PF, moon-germs-v1_main:C_0805
- added C13, C26, C33, C34, C4, C7: 2.2UF, moon-germs-v1_main:C_0805
- added C31, C32: 1.0UF, moon-germs-v1_main:C_0805
- added C36: 0.15UF, moon-germs-v1_main:C_0805
- added D5: ORANGE, moon-germs-v1_main:CHIPLED_0805
- added D6: AP7313, moon-germs-v1:SOT23-3
- added FUSE2: (no value), moon-germs-v1_main:0805
- added G3: 16MHz, moon-germs-v1_main:HC49US
- added G4: 32.768kHz, moon-germs-v1_main:TC26H
- added J5: SWITCHCRAFT_PHONEJACK, moon-germs-v1_main:STEREO_JACK_2SWITCH
- added J6: SWD_CONNECTOR, moon-germs-v1_main:1X5HEADER
- added K3: (no value), moon-germs-v1_main:LQFP64-05
- added K4: (no value), moon-germs-v1_main:LQFP32-08
- added L1, L4: (no value), moon-germs-v1_main:L0603
- added L3: FERRITE600, moon-germs-v1_main:0805
- added R11, R12: 2.2K, moon-germs-v1_main:0805
- added R13, R14: 10K, moon-germs-v1_main:0805
- added R17: 1K, moon-germs-v1_main:0805
- added R18: 100K, moon-germs-v1_main:0805
- added R5, R6: 33, moon-germs-v1_main:0805
- added R7, R8: 470, moon-germs-v1_main:0805
- added S2: (no value), moon-germs-v1_main:SWITCH_PTS820
- added T2: MCP1825S, moon-germs-v1_main:SOT-223
- added U$6: MICROSD, moon-germs-v1_main:MICRO-SD-SOCKET
- added U4: SGTL5000_32QFN, moon-germs-v1_main:QFN-32-5MM
- added U5: 23LC1024, moon-germs-v1_main:TSSOP8
- moved C1 6.35 mm to (47.0, 30.5), turned to 270 degrees
- moved D1 4.58 mm to (31.8, 27.9), turned to 270 degrees
- moved R1 4.02 mm to (31.8, 33.0), turned to 90 degrees
- moved OK1 2.84 mm to (38.1, 30.5)
- moved J3 2.84 mm to (81.3, 6.35)
- moved U$3 2.54 mm to (57.1, 39.4)
- moved R2 1.27 mm to (44.5, 30.5), turned to 90 degrees
Connections:
- removed net 5V: C1.+, OK1.8
- new net AGND: C13.-, C14.-, C27.-, K3.15, K3.16, L4.2
- new net AMPSD: J5.4, R18.2
- new net AREF: C14.+, K3.14, R8.2
- new net D+: R6.1, U$2.3
- new net D-: R5.1, U$2.2
- new net EN': J6.5, K4.7
- new net N$10: G4.1, K3.20
- new net N$11: G4.2, K3.19
- new net N$12: C12.+, G3.2, K3.33
- new net N$13: C11.+, G3.1, K3.32
- new net N$14: C13.+, K3.13, L1.1, R8.1
- new net N$15: C27.+, K3.17
- new net N$19: C36.+, U4.10
- new net N$20: C33.+, D6.OUT, U4.30
- new net N$21: C34.+, C35.+, L3.2, U4.5
- new net N$8: K3.24, K4.17
- new net N$9: D5.C, R7.2
- new net PIN0/SW1: K3.39
- new net PIN1/SW2: K3.40
- new net PIN10/DAT3: K3.49, R14.1, U$6.CS(2)
- new net PIN11/MCLK: K3.51, U4.21
- new net PIN12/DAT0: K3.52, U$6.DO(7), U5.2
- new net PIN13/RX: D5.A, K3.50, U4.25
- new net PIN14/CLK: K3.58, U$6.SCLK(5), U5.6
- new net PIN15(VOL): K3.43
- new net PIN16: K3.35
- new net PIN17: K3.36
- new net PIN18/SDA: K3.38, R12.1, U4.27
- new net PIN19/SCL: K3.37, R11.1, U4.29
- new net PIN2: K3.57
- new net PIN20/ENC_LED_G: K3.62
- new net PIN21/ENC_LED_R: K3.63
- new net PIN22/TX: K3.44, U4.26
- new net PIN23/LRCLK: K3.45, U4.23
- new net PIN24: K3.27
- new net PIN25: K3.42
- new net PIN26: K3.2
- new net PIN27: K3.54
- new net PIN28: K3.53
- new net PIN29: K3.55
- new net PIN3: K3.28
- new net PIN30: K3.56
- new net PIN31: K3.1
- new net PIN32/SW3: K3.41
- new net PIN33: K3.26
- new net PIN4/ENCA: K3.29
- new net PIN5/ENCB: K3.64
- new net PIN6/CS: K3.61, R13.2, U5.1
- new net PIN7/CMD: K3.59, U$6.DI(3), U5.5
- new net PIN8/ENCSW: K3.60
- new net PIN9/BCLK: K3.46, U4.24
- new net PINA10: K3.9
- new net PINA11: K3.10
- new net PINA12: K3.11
- new net PINA13: K3.12
- new net PINA14/MOD: K3.18
- new net PROG: K4.18, S2.1
- new net RING/R: J5.3, U4.2
- new net RST: J6.2, K3.34, K4.25, K4.8
- new net SLEEVE: J5.1, U4.4
- new net SWC: J6.4, K3.22, K4.16
- new net SWD: J6.3, K3.25, K4.15
- new net TIP/L: J5.2, R17.1, U4.6
- new net USB_DM: K3.6, R5.2
- new net USB_DP: K3.5, R6.2
- new net USB_ID: K3.23, K4.10
- new net VIN_5V: C3.+, J1.1, T2.1
- new net VUSB: FUSE2.2
- new net VUSB_IN: C4.+, FUSE2.1, U$2.1
- net 3.3V: now also C1.+, C10.+, C26.+, C28.+, C29.+, C31.+, C32.+, C7.+, C8.+, C9.+, D6.IN, K3.21, K3.3, K3.30, K3.48, K3.7, K4.3, K4.4, L1.2, L3.1, OK1.8, R11.2, R12.2, R13.1, R14.2, R17.2, T2.3, U$6.VCC(4), U4.20, U5.3, U5.7, U5.8
- net GND: now also C10.-, C11.-, C12.-, C26.-, C28.-, C29.-, C3.-, C31.-, C32.-, C33.-, C34.-, C35.-, C36.-, C4.-, C7.-, C8.-, C9.-, D6.GND, J1.2, J6.1, K3.31, K3.4, K3.47, K4.5, K4.6, L4.1, R18.1, R7.1, S2.2, T2.2, T2.PAD, U$2.4, U$6.GND(6), U4.1, U4.3, U4.31, U4.32, U4.7, U4.PAD, U5.4
Routing:
- net PIN19/SCL: track 0.00 -> 88.1 mm, vias 0 -> 4
- net PIN18/SDA: track 0.00 -> 78.7 mm, vias 0 -> 4
- net PIN22/TX: track 0.00 -> 75.0 mm, vias 0 -> 4
- net PIN23/LRCLK: track 0.00 -> 71.6 mm, vias 0 -> 2
- net PIN9/BCLK: track 0.00 -> 71.3 mm, vias 0 -> 2
- net SWC: track 0.00 -> 59.0 mm
- net GND: track 0.00 -> 35.1 mm, vias 0 -> 4
- net 3.3V: track 0.00 -> 31.5 mm
- net USB_ID: track 0.00 -> 27.2 mm
- net PIN10/DAT3: track 0.00 -> 26.8 mm
- net SWD: track 0.00 -> 26.3 mm, vias 0 -> 4
- net RST: track 0.00 -> 22.8 mm, vias 0 -> 2
- net EN': track 0.00 -> 21.6 mm
- net PIN7/CMD: track 0.00 -> 21.5 mm
- net PIN12/DAT0: track 0.00 -> 19.6 mm
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- added copper zone on layer 1, net GND
- added copper zone on layer 16, net GND

Commit message: more routing
Parts:
- moved R13 11.3 mm to (54.0, 17.8), turned to 270 degrees
- moved U5 6.02 mm to (48.9, 17.8), turned to 0 degrees
- moved R7 5.67 mm to (25.8, 12.2)
- moved R14 3.82 mm to (48.9, 14.9), turned to 180 degrees
- moved D5 1.45 mm to (23.2, 15.1)
- moved J3 1.00 mm to (81.0, 5.40), turned to 180 degrees
Connections:
- net PIN0/SW1 renamed PIN0/MIDIIN
- net PIN1/SW2 renamed PIN1/MIDIOUT
- removed net PIN15(VOL): K3.43
- removed net PIN16: K3.35
- removed net PIN17: K3.36
- removed net PIN2: K3.57
- removed net PIN20/ENC_LED_G: K3.62
- removed net PIN21/ENC_LED_R: K3.63
- removed net PIN24: K3.27
- removed net PIN25: K3.42
- removed net PIN26: K3.2
- removed net PIN27: K3.54
- removed net PIN28: K3.53
- removed net PIN29: K3.55
- removed net PIN3: K3.28
- removed net PIN30: K3.56
- removed net PIN31: K3.1
- removed net PIN32/SW3: K3.41
- removed net PIN33: K3.26
- removed net PIN4/ENCA: K3.29
- removed net PIN5/ENCB: K3.64
- removed net PIN8/ENCSW: K3.60
- removed net PINA10: K3.9
- removed net PINA11: K3.10
- removed net PINA12: K3.11
- removed net PINA13: K3.12
- removed net PINA14/MOD: K3.18
- new net PIN15/KNOB1(VOL): J3.P$5, K3.43
- new net PIN16/KNOB2: J3.P$6, K3.35
- new net PIN17/KNOB3: J3.P$7, K3.36
- new net PIN2/SW1: J3.P$1, K3.57
- new net PIN20/KNOB4: J3.P$8, K3.62
- new net PIN21/KNOB5: J3.P$9, K3.63
- new net PIN24/LED1: J3.P$22, K3.27
- new net PIN25/LED2: J3.P$23, K3.42
- new net PIN26/KNOB6: J3.P$10, K3.2
- new net PIN27/KNOB7: J3.P$11, K3.54
- new net PIN28/KNOB8: J3.P$12, K3.53
- new net PIN29/KNOB9: J3.P$13, K3.55
- new net PIN3/SW2: J3.P$2, K3.28
- new net PIN30/KNOB10: J3.P$14, K3.56
- new net PIN31/KNOB11: J3.P$15, K3.1
- new net PIN32/LED3: J3.P$24, K3.41
- new net PIN33/LED4: J3.P$25, K3.26
- new net PIN4/SW3: J3.P$3, K3.29
- new net PIN5/SW4: J3.P$4, K3.64
- new net PIN8/MIDILED: J3.P$21, K3.60
- new net PINA10/KNOB12: J3.P$16, K3.9
- new net PINA11/KNOB13: J3.P$17, K3.10
- new net PINA12/KNOB14: J3.P$18, K3.11
- new net PINA13/KNOB15: J3.P$19, K3.12
- new net PINA14/KNOB16: J3.P$20, K3.18
- net 3.3V: now also J3.P$26, J3.P$27, J3.P$28
- net GND: now also J3.P$29, J3.P$30
Routing:
- net PIN8/MIDILED: track 0.00 -> 69.9 mm
- net PIN4/SW3: track 0.00 -> 54.6 mm, vias 0 -> 1
- net PIN3/SW2: track 0.00 -> 52.9 mm, vias 0 -> 1
- net PIN24/LED1: track 0.00 -> 51.1 mm, vias 0 -> 1
- net PIN33/LED4: track 0.00 -> 49.9 mm, vias 0 -> 1
- net PIN16/KNOB2: track 0.00 -> 49.2 mm, vias 0 -> 2
- net PIN17/KNOB3: track 0.00 -> 48.4 mm, vias 0 -> 2
- net PIN32/LED3: track 0.00 -> 46.6 mm, vias 0 -> 2
- net PIN25/LED2: track 0.00 -> 45.2 mm, vias 0 -> 2
- net PIN15/KNOB1(VOL): track 0.00 -> 44.1 mm, vias 0 -> 2
- net PIN28/KNOB8: track 0.00 -> 43.3 mm, vias 0 -> 1
- net PIN27/KNOB7: track 0.00 -> 43.1 mm, vias 0 -> 1
- net PIN29/KNOB9: track 0.00 -> 42.5 mm, vias 0 -> 1
- net PIN30/KNOB10: track 0.00 -> 41.9 mm, vias 0 -> 1
- net PIN2/SW1: track 0.00 -> 41.2 mm, vias 0 -> 1
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
Commit message: lots o' routing
Parts:
- removed R17: 1K, moon-germs-v1_main:0805
- removed R18: 100K, moon-germs-v1_main:0805
- J3: device sirin-clone-library:AMPHENOL_30_PIN -> sirin-clone-library:MOLEX_30PINCONNECTOR_2MM
- moved FUSE2 90.3 mm to (7.62, 39.7), turned to 0 degrees
- moved C4 87.5 mm to (3.49, 39.7)
- moved C26 22.2 mm to (86.2, 37.9), turned to 0 degrees
- moved D6 20.4 mm to (86.4, 35.2), turned to 90 degrees
- moved C31 19.0 mm to (86.4, 32.3), turned to 0 degrees
- moved C32 15.0 mm to (86.4, 30.5)
- moved C33 11.8 mm to (81.9, 32.0), turned to 180 degrees
- moved R13 9.92 mm to (60.3, 10.2)
- moved U5 9.34 mm to (54.3, 10.2)
- moved R14 5.84 mm to (46.7, 9.53), turned to 0 degrees
- moved J3 4.14 mm to (81.3, 9.53), turned to 0 degrees
- moved C13 2.84 mm to (21.3, 34.9), turned to 180 degrees
- moved L3 2.56 mm to (71.8, 26.4), turned to 90 degrees
- moved R5 2.22 mm to (25.8, 32.0), turned to 315 degrees
- moved R8 2.08 mm to (24.4, 35.9), turned to 90 degrees
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Connections:
- removed net AMPSD: J5.4, R18.2
- new net N$27: J3.P$2
- net 3.3V: now also J3.P$14, J3.P$15; no longer J3.P$26, J3.P$27, J3.P$28, R17.2
- net GND: no longer R18.1
- net PIN15/KNOB1(VOL): now also J3.P$24; no longer J3.P$5
- net PIN16/KNOB2: now also J3.P$28; no longer J3.P$6
- net PIN17/KNOB3: now also J3.P$27; no longer J3.P$7
- net PIN2/SW1: now also J3.P$19; no longer J3.P$1
- net PIN20/KNOB4: now also J3.P$4; no longer J3.P$8
- net PIN21/KNOB5: now also J3.P$5; no longer J3.P$9
- net PIN24/LED1: now also J3.P$16; no longer J3.P$22
- net PIN25/LED2: now also J3.P$25; no longer J3.P$23
- net PIN26/KNOB6: now also J3.P$9; no longer J3.P$10
- net PIN27/KNOB7: now also J3.P$22; no longer J3.P$11
- net PIN28/KNOB8: now also J3.P$23; no longer J3.P$12
- net PIN29/KNOB9: now also J3.P$21; no longer J3.P$13
- net PIN3/SW2: now also J3.P$17; no longer J3.P$2
- net PIN30/KNOB10: now also J3.P$20; no longer J3.P$14
- net PIN31/KNOB11: now also J3.P$8; no longer J3.P$15
- net PIN32/LED3: now also J3.P$26; no longer J3.P$24
- net PIN33/LED4: now also J3.P$1; no longer J3.P$25
- net PIN4/SW3: now also J3.P$18; no longer J3.P$3
- net PIN5/SW4: now also J3.P$6; no longer J3.P$4
- net PIN8/MIDILED: now also J3.P$3; no longer J3.P$21
- net PINA10/KNOB12: now also J3.P$11; no longer J3.P$16
- net PINA11/KNOB13: now also J3.P$10; no longer J3.P$17
- net PINA12/KNOB14: now also J3.P$12; no longer J3.P$18
- net PINA13/KNOB15: now also J3.P$13; no longer J3.P$19
- net PINA14/KNOB16: now also J3.P$7; no longer J3.P$20
- net TIP/L: no longer R17.1
- net VUSB: now also U$2.1
- net VUSB_IN: no longer U$2.1
Routing:
- net 3.3V: track 31.5 -> 322.5 mm, vias 0 -> 20
- net PINA14/KNOB16: track 0.00 -> 87.7 mm, vias 0 -> 4
- net PINA10/KNOB12: track 0.00 -> 85.2 mm, vias 0 -> 4
- net PINA13/KNOB15: track 0.00 -> 82.2 mm, vias 0 -> 4
- net PINA12/KNOB14: track 0.00 -> 79.5 mm, vias 0 -> 4
- net PINA11/KNOB13: track 0.00 -> 74.4 mm, vias 0 -> 4
- net PIN13/RX: track 5.39 -> 77.3 mm, vias 0 -> 6
- net PIN26/KNOB6: track 0.00 -> 68.0 mm, vias 0 -> 2
- net PIN31/KNOB11: track 0.00 -> 64.6 mm, vias 0 -> 2
- net PIN11/MCLK: track 13.1 -> 68.6 mm, vias 1 -> 6
- net GND: track 35.4 -> 89.0 mm, vias 4 -> 22
- net PIN16/KNOB2: track 49.2 -> 102.8 mm, vias 2 -> 4
- net PIN17/KNOB3: track 48.4 -> 99.5 mm, vias 2 -> 4
- net PIN32/LED3: track 46.6 -> 95.8 mm, vias 2 -> 4
- net PIN25/LED2: track 45.2 -> 93.8 mm, vias 2 -> 4
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- added copper zone on layer 1, net AGND

Commit message: ready for gerbers
Parts:
- removed C4: 2.2UF, moon-germs-v1_main:C_0805
- removed FUSE2: (no value), moon-germs-v1_main:0805
- removed U$2: USB-B, sirin-clone-library:USB-B
- added C2, C5: 1UF, sirin-clone-library:C_0805
- added J2: (no value), sirin-clone-library:USB-MICROB-PTH-MILL
- L3: value FERRITE600 -> FER600
- R1: value 220OHM -> 220
- R2: value 470OHM -> 470
- moved J1 1.93 mm to (90.2, 45.4)
- moved U$1 1.27 mm to (33.3, 54.7)
- moved J5 0.58 mm to (72.4, 56.6)
- moved C28 0.46 mm to (9.91, 30.9)
- moved C9 0.46 mm to (12.3, 33.3)
Connections:
- removed net N$27: J3.P$2
- removed net N$4: OK1.6, R2.1
- removed net VUSB: FUSE2.2, U$2.1
- new net N$16: C5.-, U$3.6
- new net N$5: C5.+, U4.12
- new net N$6: C2.+, U4.11
- new net N$7: C2.-, U$3.5
- net AGND: now also J3.P$29, J3.P$30
- net D+: now also J2.D+; no longer U$2.3
- net D-: now also J2.D-; no longer U$2.2
- net GND: now also J2.GND, J2.SHIELD, J2.SHIELD10, J2.SHIELD2, J2.SHIELD3, J2.SHIELD4, J2.SHIELD5, J2.SHIELD6, J2.SHIELD7, J2.SHIELD8, J2.SHIELD9, J3.P$13, U$3.4; no longer C4.-, J3.P$29, J3.P$30, U$2.4
- net PIN0/MIDIIN: now also OK1.6, R2.1
- net PIN20/KNOB4: now also J3.P$3; no longer J3.P$4
- net PIN21/KNOB5: now also J3.P$4; no longer J3.P$5
- net PIN26/KNOB6: now also J3.P$8; no longer J3.P$9
- net PIN31/KNOB11: now also J3.P$7; no longer J3.P$8
- net PIN5/SW4: now also J3.P$5; no longer J3.P$6
- net PIN8/MIDILED: now also J3.P$2; no longer J3.P$3
- net PINA10/KNOB12: now also J3.P$10; no longer J3.P$11
- net PINA11/KNOB13: now also J3.P$9; no longer J3.P$10
- net PINA12/KNOB14: now also J3.P$11; no longer J3.P$12
- net PINA13/KNOB15: now also J3.P$12; no longer J3.P$13
- net PINA14/KNOB16: now also J3.P$6; no longer J3.P$7
- net USB_ID: now also J2.ID
- net VUSB_IN: now also J2.VBUS; no longer C4.+, FUSE2.1
Routing:
- net AGND: track 0.00 -> 112.3 mm, vias 0 -> 18
- net PIN0/MIDIIN: track 0.00 -> 50.5 mm, vias 0 -> 4
- net GND: track 89.0 -> 135.7 mm, vias 22 -> 23
- net USB_ID: track 27.2 -> 49.4 mm, vias 0 -> 2
- net N$16: track 0.00 -> 17.8 mm
- net N$7: track 0.00 -> 17.3 mm
- net N$6: track 0.00 -> 15.4 mm, vias 0 -> 2
- net N$5: track 0.00 -> 11.9 mm, vias 0 -> 2
- net D-: track 27.3 -> 33.5 mm, vias 0 -> 2
- net 3.3V: track 322.5 -> 326.5 mm, vias 20 -> 22
- net D+: track 29.7 -> 33.6 mm
- net N$4: track 2.70 -> 0.00 mm
- net VUSB: track 2.58 -> 0.00 mm
- net PIN8/MIDILED: track 54.9 -> 52.4 mm
- net PIN20/KNOB4: track 55.8 -> 53.5 mm
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Other:
- board text added: "EN"
- board text added: "GND"
- board text added: "MAIN BOARD V0.0.1 MAR 2019 BY K. MARUT"
- board text added: "RST"
- board text added: "SWC"
- board text added: "SWD"

Commit message: adding bom attributes
Parts:
- J2: device sirin-clone-library:USB-MICROB-PTH-MILL -> sirin-clone-library:FCI_10103594-0001LF
- moved J2 3.17 mm to (14.0, 55.2)
Connections:
- net GND: now also J2.S1, J2.S2, J2.S3, J2.S4, J2.S5, J2.S6; no longer J2.SHIELD, J2.SHIELD10, J2.SHIELD2, J2.SHIELD3, J2.SHIELD4, J2.SHIELD5, J2.SHIELD6, J2.SHIELD7, J2.SHIELD8, J2.SHIELD9
- net VUSB_IN: now also J2.VCC; no longer J2.VBUS
Routing:
- net GND: track 135.7 -> 124.8 mm, vias 23 -> 21
Other:
- board text added: "+5V IN"
- board text added: "3.3V"
- board text added: "AGND"
- board text added: "HP OUT"
- board text added: "MIDI IN"
- board text added: "PIN1"
- board text added: "PIN16"
- board text added: "STEREO LINE OUT"
- board text added: "USB MIDI"
