File: sirin-clone-schematic.sch (EAGLE design)
At the start: 21 parts

Commit message: lots o' routing
Parts:
- removed U$11: BOURNS_20K_POTENTIOMETER, sirin-clone-library:BOURNS_20K_POTENTIOMETER
- added J1: 30_PIN_CONNECTOR_MALE, sirin-clone-library:30_PIN_CONNECTOR_MALE
- added R1, R2, R3, R4: 75OHM, sirin-clone-library:75OHM
Connections:
- new net 3.3V: J1.P$14, J1.P$15, U$1.1, U$10.1, U$12.1, U$13.1, U$14.1, U$15.1, U$16.1, U$17.1, U$2.1, U$3.1, U$4.1, U$5.1, U$6.1, U$7.1, U$8.1, U$9.1
- new net GND: J1.P$29, J1.P$30, U$1.3, U$10.3, U$12.3, U$13.3, U$14.3, U$15.3, U$16.3, U$17.3, U$18.-, U$18.1, U$18.2, U$19.-, U$19.1, U$19.2, U$2.3, U$20.-, U$20.1, U$20.2, U$21.-, U$21.1, U$21.2, U$3.3, U$4.3, U$5.3, U$6.3, U$7.3, U$8.3, U$9.3
- new net N$1: R1.1, U$18.+
- new net N$2: R2.1, U$19.+
- new net N$3: R3.1, U$20.+
- new net N$4: R4.1, U$21.+
- new net PIN15/KNOB1(VOL): J1.P$24, U$13.2
- new net PIN16/KNOB2: J1.P$28, U$6.2
- new net PIN17/KNOB3: J1.P$27, U$7.2
- new net PIN2/SW1: J1.P$19, U$18.3, U$18.4
- new net PIN20/KNOB4: J1.P$4, U$8.2
- new net PIN21/KNOB5: J1.P$5, U$9.2
- new net PIN24/LED1: J1.P$16, R1.2
- new net PIN25/LED2: J1.P$25, R2.2
- new net PIN26/KNOB6: J1.P$9, U$10.2
- new net PIN27/KNOB7: J1.P$22, U$17.2
- new net PIN28/KNOB8: J1.P$23, U$12.2
- new net PIN29/KNOB9: J1.P$21, U$14.2
- new net PIN3/SW2: J1.P$17, U$19.3, U$19.4
- new net PIN30/KNOB10: J1.P$20, U$15.2
- new net PIN31/KNOB11: J1.P$8, U$1.2
- new net PIN32/LED3: J1.P$26, R3.2
- new net PIN33/LED4: J1.P$1, R4.2
- new net PIN4/SW3: J1.P$18, U$20.3, U$20.4
- new net PIN5/SW4: J1.P$6, U$21.3, U$21.4
- new net PIN8/MIDILED: J1.P$3
- new net PINA10/KNOB12: J1.P$11, U$2.2
- new net PINA11/KNOB13: J1.P$10, U$3.2
- new net PINA12/KNOB14: J1.P$12, U$4.2
- new net PINA13/KNOB15: J1.P$13, U$5.2
- new net PINA14/KNOB16: J1.P$7, U$16.2
Other:
- moved on the sheet: U$1, U$10, U$12, U$13, U$14, U$15, U$16, U$17, U$18, U$19, U$2, U$20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

Commit message: ready for gerbers
Parts:
- added D1: (no value), sirin-clone-library:LED_RED0805
- added R5: 75OHM, sirin-clone-library:75OHM
Connections:
- new net AGND: J1.P$29, J1.P$30, U$1.3, U$10.3, U$12.3, U$13.3, U$14.3, U$15.3, U$16.3, U$17.3, U$2.3, U$3.3, U$4.3, U$5.3, U$6.3, U$7.3, U$8.3, U$9.3
- new net N$6: D1.A, R5.1
- net GND: now also D1.C, J1.P$13; no longer J1.P$29, J1.P$30, U$1.3, U$10.3, U$12.3, U$13.3, U$14.3, U$15.3, U$16.3, U$17.3, U$2.3, U$3.3, U$4.3, U$5.3, U$6.3, U$7.3, U$8.3, U$9.3
- net PIN20/KNOB4: now also J1.P$3; no longer J1.P$4
- net PIN21/KNOB5: now also J1.P$4; no longer J1.P$5
- net PIN26/KNOB6: now also J1.P$8; no longer J1.P$9
- net PIN31/KNOB11: now also J1.P$7; no longer J1.P$8
- net PIN5/SW4: now also J1.P$5; no longer J1.P$6
- net PIN8/MIDILED: now also J1.P$2, R5.2; no longer J1.P$3
- net PINA10/KNOB12: now also J1.P$10; no longer J1.P$11
- net PINA11/KNOB13: now also J1.P$9; no longer J1.P$10
- net PINA12/KNOB14: now also J1.P$11; no longer J1.P$12
- net PINA13/KNOB15: now also J1.P$12; no longer J1.P$13
- net PINA14/KNOB16: now also J1.P$6; no longer J1.P$7

Commit message: adding bom attributes
Parts:
- U$1, U$10, U$12, U$13, U$14, U$15, U$16, U$17, U$2, U$3, U$4, U$5, U$6, U$7, U$8, U$9: value BOURNS_20K_POTENTIOMETER -> BOURNS_10K_POTENTIOMETER; device sirin-clone-library:BOURNS_20K_POTENTIOMETER -> sirin-clone-library:BOURNS_10K_POTENTIOMETER
Changed lines of the file:
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@@
 <setting verticaltext="up"/>
 </settings>
-<grid distance="0.05" unitdist="inch" unit="inch" style="lines" multiple="1" display="no" altdistance="0.01" altunitdist="inch" altunit="inch"/>
+<grid distance="0.1" unitdist="inch" unit="inch" style="lines" multiple="1" display="no" altdistance="0.01" altunitdist="inch" altunit="inch"/>
 <layers>
 <layer number="1" name="Top" color="4" fill="1" visible="no" active="no"/>
@@
 </classes>
 <parts>
-<part name="U$1" library="sirin-clone-library" library_urn="urn:adsk.eagle:library:9336050" deviceset="BOURNS_20K_POTENTIOMETER" device="" package3d_urn="urn:adsk.eagle:package:9336105/2"/>
-<part name="U$2" library="sirin-clone-library" library_urn="urn:adsk.eagle:library:9336050" deviceset="BOURNS_20K_POTENTIOMETER" device="" package3d_urn="urn:adsk.eagle:package:9336105/2"/>
-<part name="U$3" library="sirin-clone-library" library_urn="urn:adsk.eagle:library:9336050" deviceset="BOURNS_20K_POTENTIOMETER" device="" package3d_urn="urn:adsk.eagle:package:9336105/2"/>
-<part name="U$4" library="sirin-clone-library" library_urn="urn:adsk.eagle:library:9336050" deviceset="BOURNS_20K_POTENTIOMETER" device="" package3d_urn="urn:adsk.eagle:package:9336105/2"/>
-<part name="U$5" library="sirin-clone-library" library_urn="urn:adsk.eagle:library:9336050" deviceset="BOURNS_20K_POTENTIOMETER" device="" package3d_urn="urn:adsk.eagle:package:9336105/2"/>
-<part name="U$6" library="sirin-clone-library" library_urn="urn:adsk.eagle:library:9336050" deviceset="BOURNS_20K_POTENTIOMETER" device="" package3d_urn="urn:adsk.eagle:package:9336105/2"/>
-<part name="U$7" library="sirin-clone-library" library_urn="urn:adsk.eagle:library:9336050" deviceset="BOURNS_20K_POTENTIOMETER" device="" package3d_urn="urn:adsk.eagle:package:9336105/2"/>
-<part name="U$8" library="sirin-clone-library" library_urn="urn:adsk.eagle:library:9336050" deviceset="BOURNS_20K_POTENTIOMETER" device="" package3d_urn="urn:adsk.eagle:package:9336105/2"/>
-<part name="U$9" library="sirin-clone-library" library_urn="urn:adsk.eagle:library:9336050" deviceset="BOURNS_20K_POTENTIOMETER" device="" package3d_urn="urn:adsk.eagle:package:9336105/2"/>
-<part name="U$10" library="sirin-clone-library" library_urn="urn:adsk.eagle:library:9336050" deviceset="BOURNS_20K_POTENTIOMETER" device="" package3d_urn="urn:adsk.eagle:package:9336105/2"/>
-<part name="U$12" library="sirin-clone-library" library_urn="urn:adsk.eagle:library:9336050" deviceset="BOURNS_20K_POTENTIOMETER" device="" package3d_urn="urn:adsk.eagle:package:9336105/2"/>
-<part name="U$13" library="sirin-clone-library" library_urn="urn:adsk.eagle:library:9336050" deviceset="BOURNS_20K_POTENTIOMETER" device="" package3d_urn="urn:adsk.eagle:package:9336105/2"/>
-<part name="U$14" library="sirin-clone-library" library_urn="urn:adsk.eagle:library:9336050" deviceset="BOURNS_20K_POTENTIOMETER" device="" package3d_urn="urn:adsk.eagle:package:9336105/2"/>
-<part name="U$15" library="sirin-clone-library" library_urn="urn:adsk.eagle:library:9336050" deviceset="BOURNS_20K_POTENTIOMETER" device="" package3d_urn="urn:adsk.eagle:package:9336105/2"/>
-<part name="U$16" library="sirin-clone-library" library_urn="urn:adsk.eagle:library:9336050" deviceset="BOURNS_20K_POTENTIOMETER" device="" package3d_urn="urn:adsk.eagle:package:9336105/2"/>
-<part name="U$17" library="sirin-clone-library" library_urn="urn:adsk.eagle:library:9336050" deviceset="BOURNS_20K_POTENTIOMETER" device="" package3d_urn="urn:adsk.eagle:package:9336105/2"/>
+<part name="U$1" library="sirin-clone-library" library_urn="urn:adsk.eagle:library:9336050" deviceset="BOURNS_10K_POTENTIOMETER" device="" package3d_urn="urn:adsk.eagle:package:9336105/2"/>
+<part name="U$2" library="sirin-clone-library" library_urn="urn:adsk.eagle:library:9336050" deviceset="BOURNS_10K_POTENTIOMETER" device="" package3d_urn="urn:adsk.eagle:package:9336105/2"/>
+<part name="U$3" library="sirin-clone-library" library_urn="urn:adsk.eagle:library:9336050" deviceset="BOURNS_10K_POTENTIOMETER" device="" package3d_urn="urn:adsk.eagle:package:9336105/2"/>
+<part name="U$4" library="sirin-clone-library" library_urn="urn:adsk.eagle:library:9336050" deviceset="BOURNS_10K_POTENTIOMETER" device="" package3d_urn="urn:adsk.eagle:package:9336105/2"/>
+<part name="U$5" library="sirin-clone-library" library_urn="urn:adsk.eagle:library:9336050" deviceset="BOURNS_10K_POTENTIOMETER" device="" package3d_urn="urn:adsk.eagle:package:9336105/2"/>
+<part name="U$6" library="sirin-clone-library" library_urn="urn:adsk.eagle:library:9336050" deviceset="BOURNS_10K_POTENTIOMETER" device="" package3d_urn="urn:adsk.eagle:package:9336105/2"/>
+<part name="U$7" library="sirin-clone-library" library_urn="urn:adsk.eagle:library:9336050" deviceset="BOURNS_10K_POTENTIOMETER" device="" package3d_urn="urn:adsk.eagle:package:9336105/2"/>
+<part name="U$8" library="sirin-clone-library" library_urn="urn:adsk.eagle:library:9336050" deviceset="BOURNS_10K_POTENTIOMETER" device="" package3d_urn="urn:adsk.eagle:package:9336105/2"/>
+<part name="U$9" library="sirin-clone-library" library_urn="urn:adsk.eagle:library:9336050" deviceset="BOURNS_10K_POTENTIOMETER" device="" package3d_urn="urn:adsk.eagle:package:9336105/2"/>
+<part name="U$10" library="sirin-clone-library" library_urn="urn:adsk.eagle:library:9336050" deviceset="BOURNS_10K_POTENTIOMETER" device="" package3d_urn="urn:adsk.eagle:package:9336105/2"/>
+<part name="U$12" library="sirin-clone-library" library_urn="urn:adsk.eagle:library:9336050" deviceset="BOURNS_10K_POTENTIOMETER" device="" package3d_urn="urn:adsk.eagle:package:9336105/2"/>
+<part name="U$13" library="sirin-clone-library" library_urn="urn:adsk.eagle:library:9336050" deviceset="BOURNS_10K_POTENTIOMETER" device="" package3d_urn="urn:adsk.eagle:package:9336105/2"/>
+<part name="U$14" library="sirin-clone-library" library_urn="urn:adsk.eagle:library:9336050" deviceset="BOURNS_10K_POTENTIOMETER" device="" package3d_urn="urn:adsk.eagle:package:9336105/2"/>
+<part name="U$15" library="sirin-clone-library" library_urn="urn:adsk.eagle:library:9336050" deviceset="BOURNS_10K_POTENTIOMETER" device="" package3d_urn="urn:adsk.eagle:package:9336105/2"/>
+<part name="U$16" library="sirin-clone-library" library_urn="urn:adsk.eagle:library:9336050" deviceset="BOURNS_10K_POTENTIOMETER" device="" package3d_urn="urn:adsk.eagle:package:9336105/2"/>
+<part name="U$17" library="sirin-clone-library" library_urn="urn:adsk.eagle:library:9336050" deviceset="BOURNS_10K_POTENTIOMETER" device="" package3d_urn="urn:adsk.eagle:package:9336105/2"/>
 <part name="U$18" library="sirin-clone-library" library_urn="urn:adsk.eagle:library:9336050" deviceset="ESWITCH__YELLOW" device="" package3d_urn="urn:adsk.eagle:package:9336176/2"/>
 <part name="U$19" library="sirin-clone-library" library_urn="urn:adsk.eagle:library:9336050" deviceset="ESWITCH__YELLOW" device="" package3d_urn="urn:adsk.eagle:package:9336176/2"/>
 <part name="U$20" library="sirin-clone-library" library_urn="urn:adsk.eagle:library:9336050" deviceset="ESWITCH__YELLOW" device="" package3d_urn="urn:adsk.eagle:package:9336176/2"/>
 <part name="U$21" library="sirin-clone-library" library_urn="urn:adsk.eagle:library:9336050" deviceset="ESWITCH__YELLOW" device="" package3d_urn="urn:adsk.eagle:package:9336176/2"/>
-<part name="J1" library="sirin-clone-library" library_urn="urn:adsk.eagle:library:9336050" deviceset="30_PIN_CONNECTOR_MALE" device="" package3d_urn="urn:adsk.eagle:package:9975532/3">
+<part name="J1" library="sirin-clone-library" library_urn="urn:adsk.eagle:library:9336050" deviceset="30_PIN_CONNECTOR_MALE" device="" package3d_urn="urn:adsk.eagle:package:9975532/4">
 <attribute name="SPICEPREFIX" value="X"/>
 </part>
